File: FreetailHardware.kicad_sch (KiCad schematic)
At the start: 50 parts, among them CON1 Transducer, J1 TX, J2 REF, J3 RX, Q1 S8050, U1 Teensy3.2, U2 LMV324

Commit message: Update R12 to 56k to reduce final stage gain
Parts:
- R12: value 470k -> 56k
Changed lines of the file:
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@@
     (in_bom yes) (on_board yes)
     (property "Reference" "R12" (id 0) (at 227.33 52.07 90))
-    (property "Value" "470k" (id 1) (at 227.33 54.61 90))
+    (property "Value" "56k" (id 1) (at 227.33 54.61 90))
     (property "Footprint" "Resistor_SMD:R_0603_1608Metric_Pad0.98x0.95mm_HandSolder" (id 2) (at 227.33 52.832 90)
       (effects (font (size 1.27 1.27)) hide)
@@
     )
     (path "/00000000-0000-0000-0000-000061afa379"
-      (reference "R12") (unit 1) (value "470k") (footprint "Resistor_SMD:R_0603_1608Metric_Pad0.98x0.95mm_HandSolder")
+      (reference "R12") (unit 1) (value "56k") (footprint "Resistor_SMD:R_0603_1608Metric_Pad0.98x0.95mm_HandSolder")
     )
     (path "/00000000-0000-0000-0000-000061afc6d3"

Commit message: v1.1 Hardware sent for fabrication
Parts:
- added J4: Conn_01x03, Connector_PinHeader_2.54mm:PinHeader_1x03_P2.54mm_Vertical, symbol Connector_Generic:Conn_01x03
- added TP7: TestPoint, TestPoint:TestPoint_THTPad_D1.5mm_Drill0.7mm, symbol Connector:TestPoint
- C1, C3: symbol Device:CP1 -> Device:C_Polarized_US
- C10, C11, C2, C4, C5, C6, C7, C8, C9: footprint Capacitor_SMD:C_0603_1608Metric_Pad1.05x0.95mm_HandSolder -> Capacitor_SMD:C_0603_1608Metric_Pad1.08x0.95mm_HandSolder
- D1: symbol Device:D_x2_Serial_AKC -> Device:D_Dual_Series_AKC_Parallel
- J1, J2, J3: DNP (none) -> Y
- JP1, JP2, JP3, JP4, JP5, JP6, JP7, JP8, JP9: now left out of the parts list
- Q1: footprint Package_TO_SOT_SMD:SOT-23 -> Package_TO_SOT_SMD:SOT-23_Handsoldering
- TP1, TP2, TP3, TP4, TP5, TP6: footprint TestPoint:TestPoint_THTPad_D1.0mm_Drill0.5mm -> TestPoint:TestPoint_THTPad_D1.5mm_Drill0.7mm; now left out of the parts list
- TR1: value 10:1 step-up 7-8nH secondary -> 10:1 step-up 7-8mH secondary
- U1: footprint teensy:Teensy30_31_32_All_Pins -> transformer:Teensy32; symbol teensy:Teensy3.2 -> transformer:Teensy3.2
Connections:
- net VAA: now also J4.2 (Pin_2)
- net at CON1.1 (Pin_1), R3.2, R4.2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: now also TP7.1
- net at C2.2, C3.1, R1.1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: no longer TP1.1
- net at Q1.3 (C), TR1.6: now also TP1.1
- net V_TX: now reaches C1.1, JP1.2 (B), JP2.1 (A), R1.2
- net V_TX: now also J4.1 (Pin_1)
- net GNDA: now reaches U1.32 (AGND)
- net GNDA: now also C1.2, C10.1, C11.1, C2.1, C3.2, C5.1, C8.2, CON1.2 (Pin_2), D1.3 (A), Q1.2 (E), R14.1, R3.1, TR1.3, TR1.7 (SHIELD), TR1.8, U2.11 (V-), J4.3 (Pin_3)
- removed net GND: C1.2, C10.1, C11.1, C2.1, C3.2, C5.1, C8.2, CON1.2 (Pin_2), D1.3 (common), Q1.2 (E), R14.1, R3.1, TR1.3, TR1.7 (SHIELD), TR1.8, U1.1 (GND), U2.11 (V-)
- removed net VCOM: R15.1, R5.1, R8.1, TP6.1, U2.1, U2.10 (+), U2.12 (+), U2.5 (+)
- new net: R15.1, TP6.1, U2.1
- no-connect marks 48 -> 30
Other:
- note added: "-5.6x high pass filter"
- note removed: "-47x high pass filter"
- moved on the sheet: TP1

Commit message: Version 1.2 sent for fabrication Fix unconnected Vbias Mark soldered pads for Teensy Add capacitor for TX filter
Parts:
- added C12: Cfilt, Capacitor_SMD:C_0603_1608Metric_Pad1.08x0.95mm_HandSolder, symbol Device:C
Connections:
- net GNDA: now also C12.2
- net Vbias: now reaches R5.1
- net Vbias: now also R15.1, R8.1, TP6.1, U2.1, U2.10 (+), U2.12 (+), U2.5 (+)
- net at Q1.1 (B), R2.2: now also C12.1
Other:
- moved on the sheet: R2
